File: PiPico_game_board.kicad_pcb (KiCad board)
At the start: 2 copper layers, 17 parts, among them U1 Pico

Commit message: Minor schematic changes
Connections:
- RV1 pad 1: 3V3 -> Net-(RV1-Pad1)
- RV1 pad 3: Net-(RV1-Pad2) -> +3V3
- SW_ACT1 pad 1: 3V3 -> +3V3
- SW_BCK1 pad 1: 3V3 -> +3V3
- SW_DWN1 pad 1: 3V3 -> +3V3
- SW_L1 pad 1: 3V3 -> +3V3
- SW_R1 pad 1: 3V3 -> +3V3
- SW_UP1 pad 1: 3V3 -> +3V3
- U1 pad 13: unconnected-(U1-Pad13) -> GND
- U1 pad 18: unconnected-(U1-Pad18) -> GND
- U1 pad 21: Net-(BZ1-Pad1) -> unconnected-(U1-Pad21)
- U1 pad 23: unconnected-(U1-Pad23) -> GND
- U1 pad 3: unconnected-(U1-Pad3) -> GND
- U1 pad 33: unconnected-(U1-Pad33) -> Net-(RV1-Pad1)
- U1 pad 36: unconnected-(U1-Pad36) -> +3V3
- U1 pad 37: 3V3 -> unconnected-(U1-Pad37)
- U1 pad 38: unconnected-(U1-Pad38) -> GND
- U1 pad 42: unconnected-(U1-Pad42) -> GND
- U1 pad 8: unconnected-(U1-Pad8) -> GND
- U1 pad 9: unconnected-(U1-Pad9) -> Net-(BZ1-Pad1)

Commit message: External power + pcb change
 - external power source
 - mounting holes
 - buttons position changed
 - changed power for OLED from VSYS to 3V3
Parts:
- removed D2, D3, D4: LED, _Easy Solder:LED_D5.0mm_Big_Pads_Back
- added BT1: Battery, _Easy Solder:BatteryWire-0.1sqmm_1x02_P3.6mm_D0.4mm_OD1mm_Relief2x_Back, F.Cu at (71.2, 107.9)
- added DP1: OLED_SPI, _Easy Solder:OLED_Display_Module, F.Cu at (74.1, 29.7)
- added D_DWN1: LED, _Easy Solder:LED_D5.0mm_Big_Pads_Back, F.Cu at (38.2, 45.0)
- added D_L1: LED, _Easy Solder:LED_D5.0mm_Big_Pads_Back, F.Cu at (45.0, 38.2)
- added D_R1: LED, _Easy Solder:LED_D5.0mm_Big_Pads_Back, F.Cu at (31.5, 38.2)
- added D_UP1: LED, _Easy Solder:LED_D5.0mm_Big_Pads_Back, F.Cu at (38.2, 31.5)
- added H1: MountingHole, MountingHole:MountingHole_2.2mm_M2, F.Cu at (29.5, 120.5)
- added H2: MountingHole, MountingHole:MountingHole_2.2mm_M2, F.Cu at (80.5, 120.5)
- added H3: MountingHole, MountingHole:MountingHole_2.2mm_M2, F.Cu at (80.5, 27.0)
- added H4: MountingHole, MountingHole:MountingHole_2.2mm_M2, F.Cu at (29.5, 27.0)
- D1: value LED -> D_Schottky; footprint _Easy Solder:LED_D5.0mm_Big_Pads_Back -> _Easy Solder:D_DO-41_SOD81_P7.62mm_Horizontal_Big_Pads_Back
- SW_DWN1, SW_L1, SW_R1, SW_UP1: footprint Button_Switch_THT:SW_PUSH_6mm -> _Easy Solder:SW_PUSH-12mm_Omron_Back
- moved SW_DWN1 218.1 mm to (52.0, 108.5), turned to -90 degrees
- moved RV1 213.8 mm to (29.0, 92.7)
- moved D1 207.2 mm to (59.5, 117.5)
- moved R3 192.8 mm to (49.0, 45.0), turned to -90 degrees
- moved SW_R1 186.8 mm to (65.0, 97.5), turned to -90 degrees
- moved SW_UP1 183.8 mm to (47.0, 99.2), turned to 90 degrees
- moved R1 179.7 mm to (45.0, 45.1), turned to -90 degrees
- moved SW_L1 176.7 mm to (39.0, 97.5), turned to -90 degrees
- moved R4 175.2 mm to (30.0, 44.8), turned to -90 degrees
- moved R2 172.5 mm to (34.2, 43.5), turned to -90 degrees
- moved SW_ACT1 161.0 mm to (80.2, 103.2), turned to 180 degrees
- moved BZ1 160.6 mm to (66.5, 43.2), turned to -90 degrees
- moved U1 158.5 mm to (52.8, 71.0), turned to 90 degrees
- moved SW_BCK1 155.8 mm to (72.0, 92.0), turned to 180 degrees
Connections:
- D1 pad 1: GND -> VSYS
- D1 pad 2: Net-(D1-Pad2) -> Net-(BT1-Pad1)
- R1 pad 1: Net-(D1-Pad2) -> Net-(D_UP1-Pad2)
- U1 pad 16: Net-(R1-Pad2) -> unconnected-(U1-Pad16)
- U1 pad 17: Net-(R2-Pad2) -> unconnected-(U1-Pad17)
- U1 pad 19: Net-(R3-Pad2) -> unconnected-(U1-Pad19)
- U1 pad 20: Net-(R4-Pad2) -> unconnected-(U1-Pad20)
- U1 pad 21: unconnected-(U1-Pad21) -> Net-(R4-Pad2)
- U1 pad 22: unconnected-(U1-Pad22) -> Net-(R3-Pad2)
- U1 pad 24: unconnected-(U1-Pad24) -> Net-(R2-Pad2)
- U1 pad 25: unconnected-(U1-Pad25) -> Net-(R1-Pad2)
Routing:
- net +3V3: track 0.00 -> 277.2 mm, vias 0 -> 6
- net GND: track 0.00 -> 140.6 mm, vias 0 -> 1
- net Net-(RV1-Pad1): track 0.00 -> 126.6 mm, vias 0 -> 3
- net Net-(RV1-Pad2): track 0.00 -> 125.4 mm, vias 0 -> 5
- net VSYS: track 0.00 -> 125.2 mm, vias 0 -> 3
- net Net-(DP1-Pad5): track 0.00 -> 74.5 mm, vias 0 -> 1
- net Net-(DP1-Pad3): track 0.00 -> 73.0 mm, vias 0 -> 1
- net Net-(DP1-Pad4): track 0.00 -> 69.9 mm, vias 0 -> 3
- net Net-(DP1-Pad6): track 0.00 -> 68.2 mm, vias 0 -> 1
- net Net-(DP1-Pad7): track 0.00 -> 67.8 mm, vias 0 -> 1
- net Net-(SW_DWN1-Pad2): track 0.00 -> 65.8 mm, vias 0 -> 1
- net Net-(BZ1-Pad1): track 0.00 -> 64.5 mm, vias 0 -> 1
- net Net-(SW_BCK1-Pad2): track 0.00 -> 60.7 mm, vias 0 -> 1
- net Net-(R4-Pad2): track 0.00 -> 58.2 mm, vias 0 -> 1
- net Net-(SW_R1-Pad2): track 0.00 -> 56.1 mm, vias 0 -> 1
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Other:
- board outline added: 56 x 98.5 mm

Commit message: Minor pcb routing changes
Routing:
- net Net-(R3-Pad2): track 32.5 -> 39.3 mm
- net Net-(R1-Pad2): track 27.3 -> 31.4 mm
- net Net-(R4-Pad2): track 58.2 -> 61.7 mm
- net Net-(R2-Pad2): track 43.6 -> 46.6 mm
- net Net-(BZ1-Pad1): track 64.5 -> 66.3 mm

Commit message: update
Parts:
- added J1: Conn_01x08, Connector_PinHeader_2.54mm:PinHeader_1x08_P2.54mm_Vertical, F.Cu at (82.2, 91.7)
- added Ref**: Val**, logo:DDM_06_F.SilkS, F.Cu at (45.5, 27.8)
- SW_ACT1, SW_BCK1: footprint Button_Switch_THT:SW_PUSH_6mm -> _Easy Solder:SW_PUSH_6mm_Back
- moved SW_ACT1 6.80 mm to (78.2, 96.8), turned to -90 degrees
- moved R4 1.24 mm to (29.9, 43.6)
- moved H2 1.00 mm to (81.5, 120.5)
- moved H3 1.00 mm to (81.5, 27.0)
- moved R1 0.59 mm to (45.0, 44.5)
- moved D1 0.50 mm to (59.0, 117.5)
- moved R3 0.50 mm to (49.0, 44.5)
- moved R2 0.34 mm to (34.1, 43.2)
- moved DP1 0.16 mm to (74.1, 29.5)
Connections:
- RV1 pad 1: Net-(RV1-Pad1) -> +3V3
- RV1 pad 3: +3V3 -> GND
- U1 pad 16: unconnected-(U1-Pad16) -> GP12
- U1 pad 17: unconnected-(U1-Pad17) -> GP13
- U1 pad 19: unconnected-(U1-Pad19) -> GP14
- U1 pad 20: unconnected-(U1-Pad20) -> GP15
- U1 pad 31: unconnected-(U1-Pad31) -> GP26
- U1 pad 32: unconnected-(U1-Pad32) -> GP27
- U1 pad 33: Net-(RV1-Pad1) -> GND
Routing:
- net Net-(RV1-Pad1): track 126.6 -> 0.00 mm, vias 3 -> 0
- net GP27: track 0.00 -> 45.0 mm
- net +3V3: track 277.2 -> 321.1 mm, vias 6 -> 7
- net GP26: track 0.00 -> 41.4 mm
- net GP12: track 0.00 -> 25.1 mm, vias 0 -> 3
- net Net-(RV1-Pad2): track 125.4 -> 100.6 mm, vias 5 -> 3
- net GP13: track 0.00 -> 22.3 mm, vias 0 -> 3
- net GP14: track 0.00 -> 15.1 mm, vias 0 -> 1
- net GP15: track 0.00 -> 14.6 mm, vias 0 -> 1
- net GND: track 140.6 -> 150.7 mm, vias 1 -> 2
- net VSYS: track 125.2 -> 120.4 mm
- net Net-(SW_DWN1-Pad2): track 65.8 -> 68.2 mm
- net Net-(SW_BCK1-Pad2): track 60.7 -> 58.8 mm
- net Net-(D_DWN1-Pad2): track 13.0 -> 14.6 mm
- net Net-(R2-Pad2): track 46.6 -> 48.2 mm
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Other:
- board size 56 x 98.5 mm -> 57 x 98.5 mm
- board text added: "1.8V-5.5V"
- board text added: "3V3"
- board text added: "DDM OLOMOUC"
- board text added: "GND"
- board text added: "GP12"
- board text added: "GP13"
- board text added: "GP14"
- board text added: "GP15"
- board text added: "GP26"
- board text added: "GP27"
- board text added: "Pi Pico Game Board"
- board text added: "v1.0 05/2022"

Commit message: Fixed previous problems + support for LCD
Parts:
- added DP2: LCD_DISPLAY_ST7735, _Easy Solder:LCD_Display_1.77_Module, F.Cu at (80.6, 48.0)
- moved R4 0.42 mm to (29.9, 43.2)
- renumbered D_R1 to D_L1, D_L1 to D_R1
Routing:
- net +3V3: track 321.1 -> 374.7 mm, vias 7 -> 10
- net GND: track 150.7 -> 182.1 mm
- net Net-(DP1-Pad5): track 74.7 -> 88.5 mm, vias 1 -> 2
- net Net-(DP1-Pad6): track 68.3 -> 80.7 mm, vias 1 -> 3
- net Net-(DP1-Pad3): track 72.9 -> 81.6 mm
- net Net-(DP1-Pad7): track 67.9 -> 72.6 mm
- net Net-(DP1-Pad4): track 70.6 -> 74.9 mm
- net Net-(R1-Pad2): track 31.2 -> 27.6 mm
- net Net-(R4-Pad2): track 60.5 -> 58.1 mm
- net Net-(R2-Pad2): track 48.2 -> 46.1 mm
- net Net-(R3-Pad2): track 38.8 -> 36.8 mm
- net Net-(BZ1-Pad1): track 66.1 -> 64.5 mm
- net GP27: track 45.0 -> 45.8 mm, vias 0 -> 2
- net GP26: track 41.4 -> 41.9 mm
Other:
- board text added: "CS"
- board text added: "D/C"
- board text added: "LCD"
- board text added: "LEDA"
- board text added: "OLED"
- board text added: "RES"
- board text added: "SCLK"
- board text added: "SDA"
- board text added: "v1.1 03/2023"
- board text removed: "v1.0 05/2022"
